Commit message: fix(urdf): replace box geometry with cylinder for base link and update inertia values

File: src/occlusion_sim/urdf/simple_holonomic_robot.urdf (robot description, URDF)
Before this commit: robot simple_holonomic_robot, 1 links, 0 joints
Links:
- link base_link: geometry collision cylinder length=0.2 radius=0.25; visual cylinder length=0.2 radius=0.25
