Commit message: feat: add arrow link and joint for direction visualization in the ego robot

File: src/occlusion_sim/urdf/simple_holonomic_robot.urdf (robot description, URDF)
Before this commit: robot simple_holonomic_robot, 1 links, 0 joints
Links:
- added link arrow; visual cylinder length=0.2 radius=0.02
Joints:
- added joint arrow_joint: type fixed, parent base_link, child arrow, origin xyz=0 0 0.15 rpy=0 0 0

Commit message: feat: add sensor visualizer node and RViz configuration for obstacle visualization

File: src/occlusion_sim/urdf/simple_holonomic_robot.urdf (robot description, URDF)
Before this commit: robot simple_holonomic_robot, 2 links, 1 joints
Links:
- removed link arrow
Joints:
- removed joint arrow_joint
